Commit message: added robot velocity controller

File: src/acrome_mini_robot/urdf/acrome_mini_robot.xacro.urdf (robot description, URDF)
Before this commit: robot acrome_mini_robot, 6 links, 5 joints
Links:
- removed link imu
- removed link world
- added link imu_link, mass 0.001; visual box size=0.01 0.01 0.01
Joints:
- removed joint world_to_base
- joint base_to_imu: child imu -> imu_link; origin xyz=0.0 0.0 0.1 -> xyz=0.0 0.0 0.15

Commit message: added our robot stl

File: src/acrome_mini_robot/urdf/acrome_mini_robot.xacro.urdf (robot description, URDF)
Before this commit: robot acrome_mini_robot, 4 links, 3 joints
Links:
- link base_link: geometry collision cylinder length=0.15 radius=0.25; visual mesh filename=file:///home/halit/acrome_ws/src/acrome_mini_robot/meshes/b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 scale=1 1 1
- link wheel_1: mass 0.5 -> 0.35; geometry collision sphere length=0.025 radius=0.025; visual sphere radius=0.015
- link wheel_2: mass 0.5 -> 0.25; geometry collision cylinder length=0.02 radius=0.04; visual mesh filename=file:///home/halit/acrome_ws/src/acrome_mini_robot/meshes/l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 scale=0.5 0.5 0.5
- link wheel_3: mass 0.5 -> 0.25; geometry collision cylinder length=0.02 radius=0.04; visual mesh filename=file:///home/halit/acrome_ws/src/acrome_mini_robot/meshes/r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 scale=0.5 0.5 0.5
Joints:
- joint base_to_wheel_1: origin xyz=0.2 0 0 rpy=0 0 0 -> xyz=0.05 0 0.05 rpy=0 0 0
- joint base_to_wheel_2: axis 0 1 0 -> 1 0 0; origin xyz=-0.1 0.173 0 rpy=0 0 2.094 -> xyz=-0.05 0.1 0 rpy=0 0 -1.5708
- joint base_to_wheel_3: axis 0 1 0 -> 1 0 0; origin xyz=-0.1 -0.173 0 rpy=0 0 -2.094 -> xyz=-0.05 -0.1 0 rpy=0 0 -1.5708

Commit message: ready to control from python

File: src/acrome_mini_robot/urdf/acrome_mini_robot.xacro.urdf (robot description, URDF)
Before this commit: robot acrome_mini_robot, 4 links, 3 joints
Links:
- link wheel_2: geometry collision cylinder length=0.02 radius=0.04; visual mesh filename=file:///home/halit/acrome_ws/src/acrome_mini_robot/meshes/l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 scale=0.7 0.7 0.7
- link wheel_3: geometry collision cylinder length=0.02 radius=0.04; visual mesh filename=file:///home/halit/acrome_ws/src/acrome_mini_robot/meshes/r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 scale=0.7 0.7 0.7
Joints:
- joint base_to_wheel_1: origin xyz=0.05 0 0.05 rpy=0 0 0 -> xyz=0.07 0 0.04 rpy=0 0 0
- joint base_to_wheel_2: origin xyz=-0.05 0.1 0 rpy=0 0 -1.5708 -> xyz=0 0.125 0.035 rpy=0 0 -1.5708
- joint base_to_wheel_3: origin xyz=-0.05 -0.1 0 rpy=0 0 -1.5708 -> xyz=0 -0.125 0.035 rpy=0 0 -1.5708
