Commit message: some little changes

File: install/acrome_mini_robot/share/acrome_mini_robot/urdf/acrome_mini_robot.xacro (robot description, xacro)
@@ -1 +1,300 @@
-/home/halit/acrome_ws/src/acrome_mini_robot/urdf/acrome_mini_robot.xacro
+<?xml version="1.0"?>
+<robot name="acrome_mini_robot" xmlns:xacro="http://www.ros.org/wiki/xacro">
+  <!-- Parametreler -->
+  <xacro:property name="lidar_radius" value="0.03"/>
+  <xacro:property name="lidar_height" value="0.04"/>
+  <xacro:property name="lidar_mass" value="0.2"/>
+  <xacro:property name="PI" value="3.141592653589793"/>
+  <!-- Ana robot gövdesi -->
+  <link name="base_link">
+    <visual>
+      <geometry>
+        <mesh filename="file:///home/halit/acrome_ws/src/acrome_mini_robot/meshes/base_link.stl" scale="1 1 1"/>
+      </geometry>
+      <origin xyz="0 0 0.075" rpy="0 0 -1.5708"/>
+      <material name="blue">
+        <color rgba="0.2 0.2 0.8 1"/>
+      </material>
+    </visual>
+    <collision>
+      <geometry>
+        <cylinder radius="0.25" length="0.15"/>
+      </geometry>
+      <origin xyz="0 0 0.075" rpy="0 0 -1.5708"/>
+    </collision>
+    <inertial>
+      <mass value="5.0"/>
+      <origin xyz="0 0 0.075" rpy="0 0 0"/>
+      <inertia ixx="0.2083" ixy="0.0" ixz="0.0" iyy="0.2083" iyz="0.0" izz="0.3125"/>
+    </inertial>
+  </link>
+  <!-- Lidar -->
+  <link name="lidar_link">
+    <visual>
+      <geometry>
+        <cylinder radius="${lidar_radius}" length="${lidar_height}"/>
+      </geometry>
+      <origin xyz="0 0 0" rpy="0 0 0"/>
+      <material name="gray"><color rgba="0.5 0.5 0.5 1"/></material>
+    </visual>
+    <collision>
+      <geometry>
+        <cylinder radius="${lidar_radius}" length="${lidar_height}"/>
+      </geometry>
+      <origin xyz="0 0 0" rpy="0 0 0"/>
+    </collision>
+    <inertial>
+      <mass value="${lidar_mass}"/>
+      <origin xyz="0 0 0" rpy="0 0 0"/>
+      <inertia ixx="0.0001" ixy="0" ixz="0" iyy="0.0001" iyz="0" izz="0.0001"/>
+    </inertial>
+  </link>
+  <!-- Caster Wheel Support (Destek Çubuğu) -->
+  <link name="caster_support">
+    <visual>
+      <geometry>
+        <cylinder radius="0.005" length="0.03"/>
+      </geometry>
+      <origin xyz="0 0 -0.015" rpy="0 0 0"/>
+      <material name="gray">
+        <color rgba="0.5 0.5 0.5 1"/>
+      </material>
+    </visual>
+    <collision>
+      <geometry>
+        <cylinder radius="0.005" length="0.03"/>
+      </geometry>
+      <origin xyz="0 0 -0.015" rpy="0 0 0"/>
+    </collision>
+    <inertial>
+      <mass value="0.05"/>
+      <origin xyz="0 0 -0.015" rpy="0 0 0"/>
+      <inertia ixx="0.00001" ixy="0" ixz="0" iyy="0.00001" iyz="0" izz="0.00001"/>
+    </inertial>
+  </link>
+  <!-- Caster Wheel -->
+  <link name="caster_wheel">
+    <visual>
+      <geometry>
+        <sphere radius="0.02"/>
+      </geometry>
+      <origin xyz="0 0 0" rpy="0 0 0"/>
+      <material name="black">
+        <color rgba="0.1 0.1 0.1 1"/>
+      </material>
+    </visual>
+    <collision>
+      <geometry>
+        <sphere radius="0.02"/>
+      </geometry>
+      <origin xyz="0 0 0" rpy="0 0 0"/>
+    </collision>
+    <inertial>
+      <mass value="0.1"/>
+      <origin xyz="0 0 0" rpy="0 0 0"/>
+      <inertia ixx="0.000016" ixy="0" ixz="0" iyy="0.000016" iyz="0" izz="0.000016"/>
+    </inertial>
+  </link>
+  <!-- Tekerlek 2 -->
+  <link name="wheel_2">
+    <visual>
+      <geometry>
+        <mesh filename="file:///home/halit/acrome_ws/src/acrome_mini_robot/meshes/left_wheel.stl" scale="0.7 0.7 0.7"/>
+      </geometry>
+      <origin xyz="0 0 0" rpy="1.5708 0 0"/>
+      <material name="black">
+        <color rgba="0.1 0.1 0.1 1"/>
+      </material>
+    </visual>
+    <collision>
+      <surface>
+        <friction>
+          <ode>
+            <mu>1.0</mu>
+            <mu2>1.0</mu2>
+          </ode>
+        </friction>
+      </surface>
+      <geometry>
+        <cylinder radius="0.06" length="0.025"/>
+      </geometry>
+      <origin xyz="0 0 0" rpy="1.5708 0 0"/>
+    </collision>
+    <inertial>
+      <mass value="0.25"/>
+      <origin xyz="0 0 0" rpy="0 0 0"/>
+      <inertia ixx="0.00045" ixy="0.0" ixz="0.0" iyy="0.00045" iyz="0.0" izz="0.00045"/>
+    </inertial>
+  </link>
+  <!-- Tekerlek 3 - Düzeltilmiş -->
+  <link name="wheel_3">
+    <visual>
+      <geometry>
+        <mesh filename="file:///home/halit/acrome_ws/src/acrome_mini_robot/meshes/right_wheel.stl" scale="0.7 0.7 0.7"/>
+      </geometry>
+      <origin xyz="0 0 0" rpy="1.5708 0 0"/>
+      <material name="black">
+        <color rgba="0.1 0.1 0.1 1"/>
+      </material>
+    </visual>
+    <collision>
+      <geometry>
+        <cylinder radius="0.06" length="0.025"/>
+      </geometry>
+      <origin xyz="0 0 0" rpy="1.5708 0 0"/>
+    </collision>
+    <inertial>
+      <mass value="0.25"/>
+      <origin xyz="0 0 0" rpy="0 0 0"/>
+      <inertia ixx="0.00045" ixy="0.0" ixz="0.0" iyy="0.00045" iyz="0.0" izz="0.00045"/>
+    </inertial>
+  </link>
+  <joint name="base_to_lidar" type="fixed">
+    <parent link="base_link"/>
+    <child link="lidar_link"/>
+    <origin xyz="0 0.0065 0.13" rpy="0 0 0"/>
+  </joint>
+  <joint name="base_to_caster_support" type="fixed">
+    <parent link="base_link"/>
+    <child link="caster_support"/>
+    <origin xyz="0.085 0 0.05" rpy="0 0 0"/>
+  </joint>
+  <joint name="caster_support_to_wheel" type="continuous">
+    <parent link="caster_support"/>
+    <child link="caster_wheel"/>
+    <origin xyz="0 0 -0.03" rpy="0 0 0"/>
+    <axis xyz="0 0 1"/>
+    <dynamics damping="0.001" friction="0.001"/>
+  </joint>
+  <joint name="base_to_wheel_2" type="continuous">
+    <parent link="base_link"/>
+    <child link="wheel_2"/>
+    <origin xyz="0 0.13 0.045" rpy="0 0 -1.5708"/>
+    <axis xyz="1 0 0"/>
+    <dynamics damping="0.1" friction="0.01"/>
+  </joint>
+  <joint name="base_to_wheel_3" type="continuous">
+    <parent link="base_link"/>
+    <child link="wheel_3"/>
+    <origin xyz="0 -0.13 0.045" rpy="0 0 -1.5708"/>
+    <axis xyz="1 0 0"/>
+    <dynamics damping="0.1" friction="0.01"/>
+  </joint>
+  <!-- ROS2 Control -->
+  <ros2_control name="GazeboSimSystem" type="system">
+    <hardware>
+      <plugin>gz_ros2_control/GazeboSimSystem</plugin>
+    </hardware>
+    <joint name="base_to_wheel_2">
+      <command_interface name="velocity">
+        <param name="min">-10</param>
+        <param name="max">10</param>
+      </command_interface>
+      <state_interface name="position"/>
+      <state_interface name="velocity"/>
+      <state_interface name="effort"/>
+    </joint>
+    <joint name="base_to_wheel_3">
+      <command_interface name="velocity">
+        <param name="min">-10</param>
+        <param name="max">10</param>
+      </command_interface>
+      <state_interface name="position"/>
+      <state_interface name="velocity"/>
+      <state_interface name="effort"/>
+    </joint>
+    <!-- Caster wheel state yayınlamak için dummy joint -->
+    <joint name="caster_support_to_wheel">
+      <state_interface name="position"/>
+      <state_interface name="velocity"/>
+      <state_interface name="effort"/>
+    </joint>
+  </ros2_control>
+  <!-- Gazebo pluginleri -->
+  <gazebo>
+    <plugin filename="gz_ros2_control-system" name="gz_ros2_control::GazeboSimROS2ControlPlugin">
+      <parameters>$(find acrome_mini_robot)/config/acrome_controller.yaml</parameters>
+    </plugin>
+  </gazebo>
+  <!-- Ana gövde sürtünmesini düşür -->
+  <gazebo reference="base_link">
+    <mu1>0.1</mu1>
+    <mu2>0.1</mu2>
+    <material>Gazebo/Blue</material>
+  </gazebo>
+  <!-- Gazebo Caster Support Ayarları -->
+  <gazebo reference="caster_support">
+    <mu1>0.1</mu1>
+    <mu2>0.1</mu2>
+    <material>Gazebo/Grey</material>
+  </gazebo>
+  <!-- Gazebo Caster Wheel Ayarları -->
+  <gazebo reference="caster_wheel">
+    <!-- Düşük sürtünme - kolayca kayabilir -->
+    <mu1>0.1</mu1>
+    <mu2>0.1</mu2>
+    <!-- Düşük sertlik değerleri -->
+    <kp>2000.0</kp>
+    <kd>5.0</kd>
+    <minDepth>0.001</minDepth>
+    <maxVel>1.0</maxVel>
+    <material>Gazebo/Black</material>
+  </gazebo>
+<!-- Gazebo ayarları - Lidar sensor kısmı -->
+  <gazebo reference="lidar_link">
+    <material>Gazebo/Black</material>
+    <sensor name="lidar_sensor" type="gpu_lidar">
+      <pose>0 0 0 0 0 0</pose>
+      <visualize>true</visualize>
+      <update_rate>10</update_rate>
+      <ray>
+        <scan>
+          <horizontal>
+            <samples>360</samples>
+            <resolution>1</resolution>
+            <min_angle>-${PI}</min_angle>
+            <max_angle>${PI}</max_angle>
+          </horizontal>
+          <vertical>
+            <samples>1</samples>
+            <resolution>1</resolution>
+            <min_angle>0</min_angle>
+            <max_angle>0</max_angle>
+          </vertical>
+        </scan>
+        <range>
+          <min>0.12</min>
+          <max>12.0</max>
+          <resolution>0.01</resolution>
+        </range>
+      </ray>
+      <always_on>1</always_on>
+      <topic>/scan</topic>
+      <plugin filename="gz-sim-sensors-system" name="gz::sim::systems::Sensors">
+        <ros>
+          <namespace></namespace>
+          <topic>scan</topic>
+          <frame_id>lidar_link</frame_id>
+        </ros>
+      </plugin>
+    </sensor>
+  </gazebo>
+  <gazebo reference="wheel_2">
+    <mu1>1.5</mu1>
+    <mu2>1.5</mu2>
+    <kp>2000.0</kp>
+    <kd>5.0</kd>
+    <minDepth>0.001</minDepth>
+    <maxVel>1.0</maxVel>
+    <material>Gazebo/Black</material>
+  </gazebo>
+  <gazebo reference="wheel_3">
+    <mu1>1.5</mu1>
+    <mu2>1.5</mu2>
+    <kp>2000.0</kp>
+    <kd>5.0</kd>
+    <minDepth>0.001</minDepth>
+    <maxVel>1.0</maxVel>
+    <material>Gazebo/Black</material>
+  </gazebo>
+</robot>

File: src/acrome_mini_robot/urdf/acrome_mini_robot.xacro (robot description, xacro)
@@ -108,4 +108,12 @@
     </visual>
     <collision>
+      <surface>
+        <friction>
+          <ode>
+            <mu>1.0</mu>
+            <mu2>1.0</mu2>
+          </ode>
+        </friction>
+      </surface>
       <geometry>
         <cylinder radius="0.06" length="0.025"/>
@@ -290,14 +298,3 @@
     <material>Gazebo/Black</material>
   </gazebo>
-  <surface>
-    <friction>
-      <ode>
-        <mu>1.5</mu>
-        <mu2>1.5</mu2>
-        <fdir1>0 1 0</fdir1>
-        <slip1>0.01</slip1>
-        <slip2>0.01</slip2>
-      </ode>
-    </friction>
-  </surface>
 </robot>
